Commit message: completed_urdf_converter

File: prisma_walker_isaaclab/asset/urdf/prisma_walker.urdf (robot description, URDF)
Before this commit: robot monopod, 28 links, 27 joints
Links:
- link albero_1: geometry collision cylinder length=99 radius=0.01; visual cylinder length=99 radius=0.01
Joints:
- joint alb_conn_bot_1: origin xyz=-0.047996 -9.5544E-05 -4.85 rpy=-3.1416 0 0 -> xyz=-0.047996 -9.5544E-05 -49.5 rpy=-3.1416 0 0
- joint albero_conn_retro_m2: origin xyz=0 -0.02 -4.85 rpy=1.5708 -1.5708 0 -> xyz=0 -0.02 -49.5 rpy=1.5708 -1.5708 0
- joint link_albero_1: origin xyz=4.85 0 0.02 rpy=1.5708 0 -1.5708 -> xyz=49.5 0 0.02 rpy=1.5708 0 -1.5708

Commit message: non si sa mai

File: prisma_walker_isaaclab/asset/urdf/prisma_walker.urdf (robot description, URDF)
Before this commit: robot monopod, 28 links, 27 joints
Links:
- link albero_1: geometry collision cylinder length=0.44 radius=0.01; visual cylinder length=0.44 radius=0.01
Joints:
- joint alb_conn_bot_1: origin xyz=-0.047996 -9.5544E-05 -3.17 rpy=-3.1416 0 0 -> xyz=-0.047996 -9.5544E-05 -0.22 rpy=-3.1416 0 0
- joint albero_conn_retro_m2: origin xyz=0 -0.02 -3.17 rpy=1.5708 -1.5708 0 -> xyz=0 -0.02 -0.22 rpy=1.5708 -1.5708 0
- joint link_albero_1: origin xyz=3.17 0 0.02 rpy=1.5708 0 -1.5708 -> xyz=0.22 0 0.02 rpy=1.5708 0 -1.5708
